File: BT.kicad_sch (KiCad schematic)
At the start: 11 parts

Commit message: new footprints
Parts:
- removed R? (x9): 10k, symbol Device:R
- C20: renamed from C12; footprint (none) -> Capacitor_SMD:C_1206_3216Metric
- U?: footprint RF_Module:ST_SPBTLE -> RF_Module:Microchip_RN4871
Other:
- moved on the sheet: C20

Commit message: GND fields
Parts:
- C20: value 10u -> 10uF
Other:
- company: (none) -> Piotr Zborowski, Łukasz Kus
Changed lines of the file:
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@@
   (title_block
     (title "Bluetooth module")
+    (date "2024-01-02")
+    (rev "v1.1")
+    (company "Piotr Zborowski, Łukasz Kus")
   )
   (junction (at 148.59 120.65) (diameter 0) (color 0 0 0 0)
@@
       (effects (font (size 1.27 1.27)) (justify left))
     )
-    (property "Value" "10u" (at 130.81 82.55 0)
+    (property "Value" "10uF" (at 130.81 82.55 0)
       (effects (font (size 1.27 1.27)) (justify left))
     )
