File: Buttons_Scrolls.kicad_sch (KiCad schematic)
At the start: 30 parts

Commit message: new footprints
Parts:
- C21, C22, C23, C24, C25, C26, C27, C28: footprint (none) -> Capacitor_SMD:C_0603_1608Metric
- R16: renamed from R21; value 10k -> 1k; footprint (none) -> Resistor_SMD:R_0603_1608Metric
- R17: renamed from R22; value 10k -> 1k; footprint (none) -> Resistor_SMD:R_0603_1608Metric
- R18: renamed from R23; value 10k -> 1k; footprint (none) -> Resistor_SMD:R_0603_1608Metric
- R19: renamed from R24; value 10k -> 1k; footprint (none) -> Resistor_SMD:R_0603_1608Metric
- R20: renamed from R25; value 10k -> 1k; footprint (none) -> Resistor_SMD:R_0603_1608Metric
- R21: renamed from R26; value 10k -> 1k; footprint (none) -> Resistor_SMD:R_0603_1608Metric
- R22: renamed from R27; value 10k -> 1k; footprint (none) -> Resistor_SMD:R_0603_1608Metric
- R23: renamed from R28; value 10k -> 1k; footprint (none) -> Resistor_SMD:R_0603_1608Metric
- R24: renamed from R29; value 10k -> 1k; footprint (none) -> Resistor_SMD:R_0603_1608Metric
- R25: renamed from R30; value 10k -> 1k; footprint (none) -> Resistor_SMD:R_0603_1608Metric
- R26: renamed from R31; value 10k -> 1k; footprint (none) -> Resistor_SMD:R_0603_1608Metric
- R27: renamed from R32; value 10k -> 1k; footprint (none) -> Resistor_SMD:R_0603_1608Metric
- R28: renamed from R33; value 10k -> 1k; footprint (none) -> Resistor_SMD:R_0603_1608Metric
- R29: renamed from R34; value 10k -> 1k; footprint (none) -> Resistor_SMD:R_0603_1608Metric
- R30: renamed from R35; value 10k -> 1k; footprint (none) -> Resistor_SMD:R_0603_1608Metric
- R31: renamed from R36; value 10k -> 1k; footprint (none) -> Resistor_SMD:R_0603_1608Metric
Other:
- note added: "Right Button"

Commit message: GND fields
Parts:
- C21, C22, C23, C24, C25, C26, C27, C28: value 10n -> 10nF
- R16, R17, R18, R19, R20, R21, R22, R23, R24, R25, R26, R27, R28, R29, R30, R31: value 1k -> 1kOhm
Other:
- company: (none) -> Piotr Zborowski, Łukasz Kus
Changed lines of the file:
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@@
   (title_block
     (title "Buttons and Scrolls")
+    (date "2024-01-02")
+    (rev "v1.1")
+    (company "Piotr Zborowski, Łukasz Kus")
   )
   (junction (at 73.66 66.04) (diameter 0) (color 0 0 0 0)
@@
       (effects (font (size 1.27 1.27)) (justify left))
     )
-    (property "Value" "10n" (at 185.42 134.62 0)
+    (property "Value" "10nF" (at 185.42 134.62 0)
       (effects (font (size 1.27 1.27)) (justify left))
     )
@@
       (effects (font (size 1.27 1.27)))
     )
-    (property "Value" "1k" (at 246.38 121.92 90)
+    (property "Value" "1kOhm" (at 246.38 121.92 90)
       (effects (font (size 1.27 1.27)))
     )
@@
       (effects (font (size 1.27 1.27)) (justify left))
     )
-    (property "Value" "1k" (at 168.91 115.57 0)
+    (property "Value" "1kOhm" (at 168.91 115.57 0)
       (effects (font (size 1.27 1.27)) (justify left))
     )
@@
       (effects (font (size 1.27 1.27)) (justify left))
     )
-    (property "Value" "10n" (at 99.06 82.55 0)
+    (property "Value" "10nF" (at 99.06 82.55 0)
       (effects (font (size 1.27 1.27)) (justify left))
     )
@@
       (effects (font (size 1.27 1.27)) (justify left))
     )
-    (property "Value" "1k" (at 76.2 138.43 0)
+    (property "Value" "1kOhm" (at 76.2 138.43 0)
       (effects (font (size 1.27 1.27)) (justify left))
     )
@@
       (effects (font (size 1.27 1.27)) (justify left))
     )
-    (property "Value" "10n" (at 83.82 82.55 0)
+    (property "Value" "10nF" (at 83.82 82.55 0)
       (effects (font (size 1.27 1.27)) (justify left))
     )
@@
       (effects (font (size 1.27 1.27)) (justify left))
     )
-    (property "Value" "10n" (at 99.06 166.37 0)
+    (property "Value" "10nF" (at 99.06 166.37 0)
       (effects (font (size 1.27 1.27)) (justify left))
     )
@@
       (effects (font (size 1.27 1.27)))
     )
-    (property "Value" "1k" (at 173.99 121.92 90)
+    (property "Value" "1kOhm" (at 173.99 121.92 90)
       (effects (font (size 1.27 1.27)))
     )
@@
       (effects (font (size 1.27 1.27)) (justify left))
     )
-    (property "Value" "10n" (at 83.82 166.37 0)
+    (property "Value" "10nF" (at 83.82 166.37 0)
       (effects (font (size 1.27 1.27)) (justify left))
     )
@@
       (effects (font (size 1.27 1.27)))
     )
-    (property "Value" "1k" (at 78.74 146.05 90)
+    (property "Value" "1kOhm" (at 78.74 146.05 90)
       (effects (font (size 1.27 1.27)))
     )
@@
       (effects (font (size 1.27 1.27)))
     )
-    (property "Value" "1k" (at 173.99 58.42 90)
+    (property "Value" "1kOhm" (at 173.99 58.42 90)
       (effects (font (size 1.27 1.27)))
     )
@@
       (effects (font (size 1.27 1.27)) (justify left))
     )
-    (property "Value" "1k" (at 168.91 52.07 0)
+    (property "Value" "1kOhm" (at 168.91 52.07 0)
       (effects (font (size 1.27 1.27)) (justify left))
     )
@@
       (effects (font (size 1.27 1.27)) (justify left))
     )
-    (property "Value" "10n" (at 257.81 134.62 0)
+    (property "Value" "10nF" (at 257.81 134.62 0)
       (effects (font (size 1.27 1.27)) (justify left))
     )
@@
       (effects (font (size 1.27 1.27)) (justify left))
     )
-    (property "Value" "1k" (at 66.04 54.61 0)
+    (property "Value" "1kOhm" (at 66.04 54.61 0)
       (effects (font (size 1.27 1.27)) (justify left))
     )
@@
       (effects (font (size 1.27 1.27)))
     )
-    (property "Value" "1k" (at 78.74 157.9471 90)
+    (property "Value" "1kOhm" (at 78.74 157.9471 90)
       (effects (font (size 1.27 1.27)))
     )
@@
       (effects (font (size 1.27 1.27)) (justify left))
     )
-    (property "Value" "1k" (at 241.3 115.57 0)
+    (property "Value" "1kOhm" (at 241.3 115.57 0)
       (effects (font (size 1.27 1.27)) (justify left))
     )
@@
       (effects (font (size 1.27 1.27)))
     )
-    (property "Value" "1k" (at 78.74 74.1271 90)
+    (property "Value" "1kOhm" (at 78.74 74.1271 90)
       (effects (font (size 1.27 1.27)))
     )
@@
       (effects (font (size 1.27 1.27)) (justify left))
     )
-    (property "Value" "10n" (at 185.42 71.12 0)
+    (property "Value" "10nF" (at 185.42 71.12 0)
       (effects (font (size 1.27 1.27)) (justify left))
     )
@@
       (effects (font (size 1.27 1.27)) (justify left))
     )
-    (property "Value" "1k" (at 241.3 52.07 0)
+    (property "Value" "1kOhm" (at 241.3 52.07 0)
       (effects (font (size 1.27 1.27)) (justify left))
     )
@@
       (effects (font (size 1.27 1.27)) (justify left))
     )
-    (property "Value" "1k" (at 66.04 138.43 0)
+    (property "Value" "1kOhm" (at 66.04 138.43 0)
       (effects (font (size 1.27 1.27)) (justify left))
     )
@@
       (effects (font (size 1.27 1.27)))
     )
-    (property "Value" "1k" (at 246.38 58.42 90)
+    (property "Value" "1kOhm" (at 246.38 58.42 90)
       (effects (font (size 1.27 1.27)))
     )
@@
       (effects (font (size 1.27 1.27)))
     )
-    (property "Value" "1k" (at 78.74 62.23 90)
+    (property "Value" "1kOhm" (at 78.74 62.23 90)
       (effects (font (size 1.27 1.27)))
     )
@@
       (effects (font (size 1.27 1.27)) (justify left))
     )
-    (property "Value" "1k" (at 76.2 54.61 0)
+    (property "Value" "1kOhm" (at 76.2 54.61 0)
       (effects (font (size 1.27 1.27)) (justify left))
     )
@@
       (effects (font (size 1.27 1.27)) (justify left))
     )
-    (property "Value" "10n" (at 257.81 71.12 0)
-      (effects (font (size 1.27 1.27)) (justify left))
-    )
+    (property "Value" "10nF" (at 257.81 71.12 0)
+      (effects (font (size 1.27 1.27)) (justify left))
+    )
