File: DCDCConverter_BMS.kicad_sch (KiCad schematic)
At the start: 11 parts

Commit message: new footprints
Parts:
- C? (x2): footprint Capacitor_THT:CP_Radial_D5.0mm_P2.00mm -> Capacitor_SMD:C_0603_1608Metric
- C?: footprint Capacitor_THT:CP_Radial_D5.0mm_P2.00mm -> Capacitor_SMD:C_0805_2012Metric
- R?: footprint Resistor_THT:R_Axial_DIN0207_L6.3mm_D2.5mm_P7.62mm_Horizontal -> Resistor_SMD:R_0201_0603Metric
- R?: footprint Resistor_THT:R_Axial_DIN0207_L6.3mm_D2.5mm_P7.62mm_Horizontal -> Resistor_SMD:R_2512_6332Metric
- R?: footprint Resistor_THT:R_Axial_DIN0207_L6.3mm_D2.5mm_P7.62mm_Horizontal -> Resistor_SMD:R_0805_2012Metric
Changed lines of the file:
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@@
       (effects (font (size 1.27 1.27)) (justify left))
     )
-    (property "Footprint" "Resistor_THT:R_Axial_DIN0207_L6.3mm_D2.5mm_P7.62mm_Horizontal" (at 195.072 106.68 90)
+    (property "Footprint" "Resistor_SMD:R_0201_0603Metric" (at 195.072 106.68 90)
       (effects (font (size 1.27 1.27)) hide)
     )
@@
         )
         (path "/7d5e88af-e2e7-4ac2-81bb-4bd53f941285/6e231fb2-3f93-4ea0-b19f-907da18ff2d0"
-          (reference "R5") (unit 1)
+          (reference "R12") (unit 1)
         )
       )
@@
       (effects (font (size 1.27 1.27)) (justify left))
     )
-    (property "Footprint" "Capacitor_THT:CP_Radial_D5.0mm_P2.00mm" (at 218.1352 96.52 0)
+    (property "Footprint" "Capacitor_SMD:C_0603_1608Metric" (at 218.1352 96.52 0)
       (effects (font (size 1.27 1.27)) hide)
     )
@@
         )
         (path "/7d5e88af-e2e7-4ac2-81bb-4bd53f941285/6e231fb2-3f93-4ea0-b19f-907da18ff2d0"
-          (reference "C7") (unit 1)
+          (reference "C15") (unit 1)
         )
       )
@@
         )
         (path "/7d5e88af-e2e7-4ac2-81bb-4bd53f941285/6e231fb2-3f93-4ea0-b19f-907da18ff2d0"
-          (reference "#PWR08") (unit 1)
+          (reference "#PWR027") (unit 1)
         )
       )
@@
   (symbol (lib_id "power:+BATT") (at 124.46 71.12 0) (unit 1)
     (in_bom yes) (on_board yes) (dnp no) (fields_autoplaced)
-    (property "Reference" "#PWR07" (at 124.46 74.93 0)
+    (property "Reference" "#PWR026" (at 124.46 74.93 0)
       (effects (font (size 1.27 1.27)) hide)
     )
@@
       (project "Computer Mouse"
         (path "/7d5e88af-e2e7-4ac2-81bb-4bd53f941285/6e231fb2-3f93-4ea0-b19f-907da18ff2d0"
-          (reference "#PWR07") (unit 1)
+          (reference "#PWR026") (unit 1)
         )
       )
@@
       (effects (font (size 1.27 1.27)) (justify left))
     )
-    (property "Footprint" "Capacitor_THT:CP_Radial_D5.0mm_P2.00mm" (at 61.9252 90.17 0)
+    (property "Footprint" "Capacitor_SMD:C_0603_1608Metric" (at 61.9252 90.17 0)
       (effects (font (size 1.27 1.27)) hide)
     )
@@
         )
         (path "/7d5e88af-e2e7-4ac2-81bb-4bd53f941285/6e231fb2-3f93-4ea0-b19f-907da18ff2d0"
-          (reference "C5") (unit 1)
+          (reference "C13") (unit 1)
         )
       )
@@
         )
         (path "/7d5e88af-e2e7-4ac2-81bb-4bd53f941285/6e231fb2-3f93-4ea0-b19f-907da18ff2d0"
-          (reference "U2") (unit 1)
+          (reference "U6") (unit 1)
         )
       )
@@
         )
         (path "/7d5e88af-e2e7-4ac2-81bb-4bd53f941285/6e231fb2-3f93-4ea0-b19f-907da18ff2d0"
-          (reference "#PWR015") (unit 1)
+          (reference "#PWR034") (unit 1)
         )
       )
@@
         )
         (path "/7d5e88af-e2e7-4ac2-81bb-4bd53f941285/6e231fb2-3f93-4ea0-b19f-907da18ff2d0"
-          (reference "#PWR012") (unit 1)
+          (reference "#PWR031") (unit 1)
         )
       )
@@
         )
         (path "/7d5e88af-e2e7-4ac2-81bb-4bd53f941285/6e231fb2-3f93-4ea0-b19f-907da18ff2d0"
-          (reference "#PWR09") (unit 1)
+          (reference "#PWR028") (unit 1)
         )
       )
@@
         )
         (path "/7d5e88af-e2e7-4ac2-81bb-4bd53f941285/6e231fb2-3f93-4ea0-b19f-907da18ff2d0"
-          (reference "#PWR014") (unit 1)
+          (reference "#PWR033") (unit 1)
         )
       )
@@
       (effects (font (size 1.27 1.27)) (justify left))
     )
-    (property "Footprint" "Resistor_THT:R_Axial_DIN0207_L6.3mm_D2.5mm_P7.62mm_Horizontal" (at 195.072 119.38 90)
+    (property "Footprint" "Resistor_SMD:R_2512_6332Metric" (at 195.072 119.38 90)
       (effects (font (size 1.27 1.27)) hide)
     )
@@
         )
         (path "/7d5e88af-e2e7-4ac2-81bb-4bd53f941285/6e231fb2-3f93-4ea0-b19f-907da18ff2d0"
-          (reference "R6") (unit 1)
+          (reference "R13") (unit 1)
         )
       )
@@
         )
         (path "/7d5e88af-e2e7-4ac2-81bb-4bd53f941285/6e231fb2-3f93-4ea0-b19f-907da18ff2d0"
-          (reference "#PWR011") (unit 1)
+          (reference "#PWR030") (unit 1)
         )
       )
@@
         )
         (path "/7d5e88af-e2e7-4ac2-81bb-4bd53f941285/6e231fb2-3f93-4ea0-b19f-907da18ff2d0"
-          (reference "#PWR06") (unit 1)
+          (reference "#PWR025") (unit 1)
         )
       )
@@
       (effects (font (size 1.27 1.27)) (justify left))
     )
-    (property "Footprint" "Resistor_THT:R_Axial_DIN0207_L6.3mm_D2.5mm_P7.62mm_Horizontal" (at 71.882 91.44 90)
+    (property "Footprint" "Resistor_SMD:R_0805_2012Metric" (at 71.882 91.44 90)
       (effects (font (size 1.27 1.27)) hide)
     )
@@
         )
         (path "/7d5e88af-e2e7-4ac2-81bb-4bd53f941285/6e231fb2-3f93-4ea0-b19f-907da18ff2d0"
-          (reference "R4") (unit 1)
+          (reference "R11") (unit 1)
         )
       )
@@
         )
         (path "/7d5e88af-e2e7-4ac2-81bb-4bd53f941285/6e231fb2-3f93-4ea0-b19f-907da18ff2d0"
-          (reference "#PWR013") (unit 1)
+          (reference "#PWR032") (unit 1)
         )
       )
@@
         )
         (path "/7d5e88af-e2e7-4ac2-81bb-4bd53f941285/6e231fb2-3f93-4ea0-b19f-907da18ff2d0"
-          (reference "J2") (unit 1)
+          (reference "J3") (unit 1)
         )
       )
@@
         )
         (path "/7d5e88af-e2e7-4ac2-81bb-4bd53f941285/6e231fb2-3f93-4ea0-b19f-907da18ff2d0"
-          (reference "L1") (unit 1)
+          (reference "L2") (unit 1)
         )
       )
@@
       (effects (font (size 1.27 1.27)) (justify left))
     )
-    (property "Footprint" "Capacitor_THT:CP_Radial_D5.0mm_P2.00mm" (at 155.2448 90.17 0)
+    (property "Footprint" "Capacitor_SMD:C_0805_2012Metric" (at 155.2448 90.17 0)
       (effects (font (size 1.27 1.27)) hide)
     )
@@
         )
         (path "/7d5e88af-e2e7-4ac2-81bb-4bd53f941285/6e231fb2-3f93-4ea0-b19f-907da18ff2d0"
-          (reference "C6") (unit 1)
+          (reference "C14") (unit 1)
         )
       )
@@
         )
         (path "/7d5e88af-e2e7-4ac2-81bb-4bd53f941285/6e231fb2-3f93-4ea0-b19f-907da18ff2d0"
-          (reference "#PWR010") (unit 1)
+          (reference "#PWR029") (unit 1)
         )
       )
@@
         )
         (path "/7d5e88af-e2e7-4ac2-81bb-4bd53f941285/6e231fb2-3f93-4ea0-b19f-907da18ff2d0"
-          (reference "U3") (unit 1)
-        )
-      )
+          (reference "U7") (unit 1)
+        )
+      )

Commit message: Bugfixes
Parts:
- R?: footprint Resistor_SMD:R_0201_0603Metric -> Resistor_SMD:R_0805_2012Metric
- R?: footprint Resistor_SMD:R_2512_6332Metric -> Resistor_SMD:R_0805_2012Metric
Changed lines of the file:
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@@
       (effects (font (size 1.27 1.27)) (justify left))
     )
-    (property "Footprint" "Resistor_SMD:R_0201_0603Metric" (at 195.072 106.68 90)
+    (property "Footprint" "Resistor_SMD:R_0805_2012Metric" (at 195.072 106.68 90)
       (effects (font (size 1.27 1.27)) hide)
     )
@@
       (effects (font (size 1.27 1.27)) (justify left))
     )
-    (property "Footprint" "Resistor_SMD:R_2512_6332Metric" (at 195.072 119.38 90)
-      (effects (font (size 1.27 1.27)) hide)
-    )
+    (property "Footprint" "Resistor_SMD:R_0805_2012Metric" (at 195.072 119.38 90)
+      (effects (font (size 1.27 1.27)) hide)
+    )

Commit message: GND fields
Other:
- company: (none) -> Piotr Zborowski, Łukasz Kus
Changed lines of the file:
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@@
   (title_block
     (title "BMS and 3.3V DC/DC Converter")
+    (date "2024-01-02")
+    (rev "v1.1")
+    (company "Piotr Zborowski, Łukasz Kus")
   )
   (junction (at 60.96 73.66) (diameter 0) (color 0 0 0 0)
