File: MCU.kicad_sch (KiCad schematic)
At the start: 20 parts

Commit message: new footprints
Parts:
- removed D?: LED_RGBK, LED_THT:LED_D5.0mm-4_RGB, symbol Device:LED_RGBK
- removed JP1: Jumper_3_Bridged12, symbol Jumper:Jumper_3_Bridged12
- removed Q? (x3): 2N3905, Package_TO_SOT_THT:TO-92_Inline, symbol Transistor_BJT:2N3905
- added D1: LED_ABGR, LED_THT:LED_D5.0mm-4_RGB, symbol Device:LED_ABGR
- added J1: Conn_01x05, Connector_JST:JST_EH_B5B-EH-A_1x05_P2.50mm_Vertical, symbol Connector_Generic:Conn_01x05
- added R? (x3): 220Ohm, Resistor_SMD:R_1206_3216Metric, symbol Device:R
- added U1, U3, U4: CPC1002N, Package_SO:SOP-4_3.8x4.1mm_P2.54mm, symbol Relay_SolidState:CPC1002N
- C1: renamed from C13; footprint (none) -> Capacitor_SMD:C_0805_2012Metric
- C2: renamed from C14; footprint (none) -> Capacitor_SMD:C_0805_2012Metric
- C3: renamed from C15; footprint (none) -> Capacitor_SMD:C_0805_2012Metric
- C4: renamed from C16; footprint (none) -> Capacitor_SMD:C_0805_2012Metric
- C5: renamed from C17; footprint (none) -> Capacitor_SMD:C_0805_2012Metric
- C6: renamed from C18; footprint (none) -> Capacitor_SMD:C_0603_1608Metric
- C7: renamed from C19; footprint (none) -> Capacitor_SMD:C_0603_1608Metric
- C8: renamed from C20; footprint (none) -> Capacitor_SMD:C_0805_2012Metric
- JP1: renamed from JP2; footprint (none) -> Jumper:SolderJumper-2_P1.3mm_Bridged2Bar_Pad1.0x1.5mm
- L1: renamed from L2; value L -> 27nH; footprint (none) -> Inductor_SMD:L_1210_3225Metric
- R? (x3): footprint Resistor_THT:R_Axial_DIN0207_L6.3mm_D2.5mm_P7.62mm_Horizontal -> Resistor_SMD:R_0805_2012Metric
- R?: footprint Resistor_THT:R_Axial_DIN0207_L6.3mm_D2.5mm_P7.62mm_Horizontal -> Resistor_SMD:R_1206_3216Metric
Connections:
- net +3V3: now also D1.1 (A), J1.1 (Pin_1)
- net GND: now also J1.5 (Pin_5), U1.2, U1.3, U3.2, U3.3, U4.2, U4.3
- net at R?.2: now also U4.4
- net at R?.2: now also U3.4
- net at R?.2: now also D1.4 (RK)
- net at JP1.1 (A), R?.2: now also U?.60 (BOOT0); no longer U?.7 (NRST)
- net at R?.1: now also D1.3 (GK)
- net at R?.1: now also U1.4
- net at U?.16 (PA2): now also R?.2
- net SWCLK: now reaches U?.46 (PA13)
- net SWCLK: now also J1.3 (Pin_3)
- net SWDIO: now reaches U?.49 (PA14)
- net SWDIO: now also J1.2 (Pin_2)
- net at U?.50 (PA15): now also R?.2
- net at U?.55 (PB3): now also R?.2
- net at R?.1: now also D1.2 (BK)
- new net: R?.1, U4.1
- new net: R?.1, U3.1
- new net: R?.1, U1.1
- new net NRST: J1.4 (Pin_4), U?.7 (NRST)
- no-connect marks 19 -> 17
Other:
- moved on the sheet: JP1, R?

Commit message: MCU-BT connection
Connections:
- net BT_P0_0: now also U?.50 (PA15); no longer U?.2 (PC13)
- net BT_P0_2: now also U?.39 (PC8); no longer U?.36 (PB15)
- net BT_P1_3: no longer U?.33 (PB12)
- net BT_P1_6: no longer U?.34 (PB13)
- net BT_P1_7: no longer U?.35 (PB14)
- net BT_P2_0: now also U?.43 (PA10); no longer U?.29 (PB10)
- net BT_P2_7: now also U?.40 (PC9); no longer U?.4 (PC15)
- net BT_P3_6: now also U?.52 (PC11); no longer U?.3 (PC14)
- net BT_RST: now also U?.51 (PC10); no longer U?.53 (PC12)
- net BT_RX: now also U?.53 (PC12); no longer U?.51 (PC10)
- net BT_TX: now also U?.54 (PD2); no longer U?.52 (PC11)
- net MOTION: no longer U?.41 (PA8)
- net SW7A: no longer U?.37 (PC6)
- net SW7B: no longer U?.38 (PC7)
- net at R?.2: no longer U?.16 (PA2)
- net at R?.2: no longer U?.50 (PA15)
- net at U?.55 (PB3): no longer R?.2
- no-connect marks 17 -> 13

Commit message: Other connections
Connections:
- net +BATT: now also U?.8 (PC0); no longer U?.14 (PA0)
- net BT_P0_2: now also U?.41 (PA8); no longer U?.39 (PC8)
- net BT_P1_2: now also U?.58 (PB6); no longer U?.30 (PB11)
- net BT_P1_3: now also U?.57 (PB5)
- net BT_P1_6: now also U?.55 (PB3)
- net BT_P1_7: now also U?.56 (PB4)
- net BT_P2_0: now also U?.39 (PC8); no longer U?.43 (PA10)
- net GND: now also C7.2, C8.2
- net MOTION: now also U?.61 (PB8)
- net REF: now also U?.9 (PC1); no longer U?.15 (PA1)
- net STAT: now also U?.59 (PB7); no longer U?.17 (PA3)
- net SW2: now also U?.10 (PC2); no longer U?.8 (PC0)
- net SW3: now also U?.11 (PC3); no longer U?.9 (PC1)
- net SW4A: now also U?.28 (PB2); no longer U?.24 (PC4)
- net SW4B: now also U?.27 (PB1); no longer U?.25 (PC5)
- net SW5: now also U?.26 (PB0); no longer U?.10 (PC2)
- net SW6: now also U?.29 (PB10); no longer U?.11 (PC3)
- net SW7A: now also U?.25 (PC5)
- net SW7B: now also U?.24 (PC4)
- net at R?.2: now also U?.14 (PA0)
- net at R?.2: now also U?.16 (PA2)
- net at R?.2: now also U?.15 (PA1)
- no-connect marks 13 -> 17

Commit message: Bugfixes
Parts:
- D1: footprint LED_THT:LED_D5.0mm-4_RGB -> LED_THT:LED_D5.0mm-4_RGB_Wide_Pins
Changed lines of the file:
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@@
       (effects (font (size 1.27 1.27)))
     )
-    (property "Footprint" "LED_THT:LED_D5.0mm-4_RGB" (at 241.3 110.49 0)
+    (property "Footprint" "LED_THT:LED_D5.0mm-4_RGB_Wide_Pins" (at 241.3 110.49 0)
       (effects (font (size 1.27 1.27)) hide)
     )

Commit message: GND fields
Parts:
- C1, C2, C3, C4, C5, C8: value 100n -> 100nF
- C6: value 4.7u -> 4.7uF
- C7: value 1u -> 1uF
Other:
- company: (none) -> Piotr Zborowski, Łukasz Kus
Changed lines of the file:
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@@
   (title_block
     (title "MCU and RGB backlight")
+    (date "2024-01-02")
+    (rev "v1.1")
+    (company "Piotr Zborowski, Łukasz Kus")
   )
   (junction (at 120.65 50.8) (diameter 0) (color 0 0 0 0)
@@
       (effects (font (size 1.27 1.27)) (justify left))
     )
-    (property "Value" "100n" (at 213.36 67.31 0)
+    (property "Value" "100nF" (at 213.36 67.31 0)
       (effects (font (size 1.27 1.27)) (justify left))
     )
@@
       (effects (font (size 1.27 1.27)) (justify left))
     )
-    (property "Value" "100n" (at 185.42 43.18 0)
+    (property "Value" "100nF" (at 185.42 43.18 0)
       (effects (font (size 1.27 1.27)) (justify left))
     )
@@
       (effects (font (size 1.27 1.27)) (justify left))
     )
-    (property "Value" "4.7u" (at 247.65 43.18 0)
+    (property "Value" "4.7uF" (at 247.65 43.18 0)
       (effects (font (size 1.27 1.27)) (justify left))
     )
@@
       (effects (font (size 1.27 1.27)) (justify left))
     )
-    (property "Value" "1u" (at 200.66 67.31 0)
+    (property "Value" "1uF" (at 200.66 67.31 0)
       (effects (font (size 1.27 1.27)) (justify left))
     )
@@
       (effects (font (size 1.27 1.27)) (justify left))
     )
-    (property "Value" "100n" (at 210.82 43.18 0)
+    (property "Value" "100nF" (at 210.82 43.18 0)
       (effects (font (size 1.27 1.27)) (justify left))
     )
@@
       (effects (font (size 1.27 1.27)) (justify left))
     )
-    (property "Value" "100n" (at 223.52 43.18 0)
+    (property "Value" "100nF" (at 223.52 43.18 0)
       (effects (font (size 1.27 1.27)) (justify left))
     )
@@
       (effects (font (size 1.27 1.27)) (justify left))
     )
-    (property "Value" "100n" (at 198.12 43.18 0)
+    (property "Value" "100nF" (at 198.12 43.18 0)
       (effects (font (size 1.27 1.27)) (justify left))
     )
@@
       (effects (font (size 1.27 1.27)) (justify left))
     )
-    (property "Value" "100n" (at 236.22 43.18 0)
-      (effects (font (size 1.27 1.27)) (justify left))
-    )
+    (property "Value" "100nF" (at 236.22 43.18 0)
+      (effects (font (size 1.27 1.27)) (justify left))
+    )
