File: OpticalSensor.kicad_sch (KiCad schematic)
At the start: 8 parts

Commit message: new footprints
Parts:
- removed Q?: 2N3905, Package_TO_SOT_THT:TO-92_Inline, symbol Transistor_BJT:2N3905
- added R?: 220Ohm, Resistor_SMD:R_1206_3216Metric, symbol Device:R
- added U9: CPC1002N, Package_SO:SOP-4_3.8x4.1mm_P2.54mm, symbol Relay_SolidState:CPC1002N
- C? (x2): footprint Capacitor_THT:CP_Radial_D5.0mm_P2.00mm -> Capacitor_SMD:C_0805_2012Metric
- C?: footprint Capacitor_THT:CP_Radial_D5.0mm_P2.00mm -> Capacitor_SMD:C_0603_1608Metric
- C?: footprint Capacitor_THT:C_Disc_D6.0mm_W2.5mm_P5.00mm -> Capacitor_SMD:C_0805_2012Metric
- R?: value 80Ohm -> 100Ohm; footprint Resistor_THT:R_Axial_DIN0207_L6.3mm_D2.5mm_P7.62mm_Horizontal -> Resistor_SMD:R_0805_2012Metric
Connections:
- net +3V3: now also U9.4
- net GND: now also U9.2
- net at R?.1: now also U9.3
- net at U?.8 (XYLED): now also R?.1
- new net: R?.2, U9.1
Other:
- moved on the sheet: D?, R?

Commit message: GND fields
Other:
- company: (none) -> Piotr Zborowski, Łukasz Kus
Changed lines of the file:
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@@
   (title_block
     (title "Optical sensor")
+    (date "2024-01-02")
+    (rev "v1.1")
+    (company "Piotr Zborowski, Łukasz Kus")
   )
   (junction (at 149.86 72.39) (diameter 0) (color 0 0 0 0)
