File: usb.kicad_sch (KiCad schematic)
At the start: 11 parts, among them U1 USBLC6-2SC6

Commit message: new footprints
Parts:
- C10: renamed from C2; footprint (none) -> Capacitor_SMD:C_0805_2012Metric
- C11: renamed from C3; footprint (none) -> Capacitor_SMD:C_0603_1608Metric
- C12: renamed from C4; footprint (none) -> Capacitor_SMD:C_0805_2012Metric
- C9: renamed from C1; footprint (none) -> Capacitor_SMD:C_0603_1608Metric
- F1: value 700m -> 750m; footprint (none) -> Fuse:Fuse_0402_1005Metric
- FB1: footprint (none) -> Capacitor_SMD:C_2220_5650Metric
- R10: renamed from R3; footprint (none) -> Resistor_SMD:R_0201_0603Metric
- R? (x2): footprint Resistor_THT:R_Axial_DIN0207_L6.3mm_D2.5mm_P7.62mm_Horizontal -> Resistor_SMD:R_0603_1608Metric
- renumbered U1 to U5

Commit message: Bugfixes
Parts:
- R10: footprint Resistor_SMD:R_0201_0603Metric -> Resistor_SMD:R_1206_3216Metric
Changed lines of the file:
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@@
       (effects (font (size 1.27 1.27)))
     )
-    (property "Footprint" "Resistor_SMD:R_0201_0603Metric" (at 62.23 121.412 90)
+    (property "Footprint" "Resistor_SMD:R_1206_3216Metric" (at 62.23 121.412 90)
       (effects (font (size 1.27 1.27)) hide)
     )

Commit message: 3.3V paths, new usb module
Parts:
- J?: footprint Connector_USB:USB_C_Receptacle_GCT_USB4105-xx-A_16P_TopMnt_Horizontal -> Connector_USB:USB_C_Receptacle_HRO_TYPE-C-31-M-12
Changed lines of the file:
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@@
       (effects (font (size 1.27 1.27)))
     )
-    (property "Footprint" "Connector_USB:USB_C_Receptacle_GCT_USB4105-xx-A_16P_TopMnt_Horizontal" (at 69.85 93.98 0)
+    (property "Footprint" "Connector_USB:USB_C_Receptacle_HRO_TYPE-C-31-M-12" (at 69.85 93.98 0)
       (effects (font (size 1.27 1.27)) hide)
     )

Commit message: GND fields
Parts:
- C10: value 100n -> 100nF
- C11: value 4.7u -> 4.7uF
- C12: value 4.7n -> 4.7nF
- C9: value 10n -> 10nF
- F1: value 750m -> 750mA
- R10: value 1M -> 1MOhm
Other:
- company: (none) -> Piotr Zborowski, Łukasz Kus
Changed lines of the file:
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@@
   (title_block
     (title "USB port")
+    (date "2024-01-02")
+    (rev "v1.1")
+    (company "Piotr Zborowski, Łukasz Kus")
   )
   (junction (at 66.04 128.27) (diameter 0) (color 0 0 0 0)
@@
       (effects (font (size 1.27 1.27)))
     )
-    (property "Value" "4.7u" (at 218.44 91.44 90)
+    (property "Value" "4.7uF" (at 218.44 91.44 90)
       (effects (font (size 1.27 1.27)))
     )
@@
       (effects (font (size 1.27 1.27)))
     )
-    (property "Value" "100n" (at 205.74 91.44 90)
+    (property "Value" "100nF" (at 205.74 91.44 90)
       (effects (font (size 1.27 1.27)))
     )
@@
       (effects (font (size 1.27 1.27)))
     )
-    (property "Value" "10n" (at 186.69 91.44 90)
+    (property "Value" "10nF" (at 186.69 91.44 90)
       (effects (font (size 1.27 1.27)))
     )
@@
       (effects (font (size 1.27 1.27)))
     )
-    (property "Value" "1M" (at 62.23 119.38 90)
+    (property "Value" "1MOhm" (at 62.23 119.38 90)
       (effects (font (size 1.27 1.27)))
     )
@@
       (effects (font (size 1.27 1.27)))
     )
-    (property "Value" "4.7n" (at 62.23 133.35 90)
+    (property "Value" "4.7nF" (at 62.23 133.35 90)
       (effects (font (size 1.27 1.27)))
     )
@@
       (effects (font (size 1.27 1.27)) (justify left))
     )
-    (property "Value" "750m" (at 228.6 76.2 90)
+    (property "Value" "750mA" (at 228.6 76.2 90)
       (effects (font (size 1.27 1.27)) (justify left))
     )
